File: Electronics/main_board_schematic_2/_restore_backup_2026-08-20T12-24-29-284/main_board_schematic_2.kicad_pcb (KiCad board)
At the start: 2 copper layers, 4 parts, among them U1 DEVKIT_V1_ESP32-WROOM-32, U2 L7805

Commit message: start kicad version of board
Parts:
- removed U2: L7805, Package_TO_SOT_THT:TO-220F-3_Horizontal_TabDown
